Commit message: Add timed simulation actions and reference geometry
Make reusable motion sequences backend-neutral and align the generated arm model with the supplied dimensions.

Co-authored-by: Cursor <cursoragent@cursor.com>

File: models/butter_finger_simple.urdf (robot description, URDF)
Before this commit: robot butter_finger, 6 links, 5 joints
Links:
- link base_link: geometry collision cylinder length=0.03253 radius=0.045; visual cylinder length=0.03253 radius=0.045
- link forearm_link: geometry collision box size=0.035 0.035 0.1; visual box size=0.035 0.035 0.1
- link turret_link: geometry collision cylinder length=0.04137 radius=0.02; visual cylinder length=0.04137 radius=0.02
- link upper_arm_link: geometry collision box size=0.035 0.035 0.1452; visual box size=0.035 0.035 0.1452
- link wrist_link: geometry collision box size=0.035 0.035 0.049; visual box size=0.035 0.035 0.049
Joints:
- joint base_joint: origin xyz=0 0 0.05 rpy=0 0 0 -> xyz=0 0 0.03253 rpy=0 0 0
- joint camera_joint: origin xyz=0 0 0.05 rpy=0 0 0 -> xyz=0 0 0.049 rpy=0 0 0
- joint elbow_joint: origin xyz=0 0 0.12 rpy=0 0 0 -> xyz=0 0 0.1452 rpy=0 0.85 0
- joint shoulder_joint: origin xyz=0 0 0.02 rpy=0 0 0 -> xyz=0 0 0.04137 rpy=0 0 0
- joint wrist_joint: origin xyz=0 0 0.12 rpy=0 0 0 -> xyz=0 0 0.1 rpy=0 0.25 0

Commit message: Add CAD-based model and simulated wrist camera
Replace primitive geometry with the recovered CAD export and add config-driven RGB camera rendering, examples, documentation, and tests.

Co-authored-by: Cursor <cursoragent@cursor.com>

File: models/butter_finger_simple.urdf (robot description, URDF)
Before this commit: robot butter_finger, 6 links, 5 joints
Links:
- link base_link: mass 0.3 -> 0.117956347342971; geometry collision mesh filename=meshes/base_link.stl; visual mesh filename=meshes/base_link.stl
- link camera_link: mass 0.01 -> 0.000001; geometry 
- link forearm_link: mass 0.08 -> 0.0294574375311473; geometry collision mesh filename=meshes/forearm_link.stl; visual mesh filename=meshes/forearm_link.stl
- link turret_link: mass 0.05 -> 0.136250635109382; geometry collision mesh filename=meshes/turret_link.stl; visual mesh filename=meshes/turret_link.stl
- link upper_arm_link: mass 0.08 -> 0.0827380990614375; geometry collision mesh filename=meshes/upper_arm_link.stl; visual mesh filename=meshes/upper_arm_link.stl
- link wrist_link: mass 0.04 -> 0.0181766061397578; geometry collision mesh filename=meshes/wrist_link.stl; visual mesh filename=meshes/wrist_link.stl
Joints:
- joint base_joint: axis 0 0 1 -> 1 0 0; origin xyz=0 0 0.03253 rpy=0 0 0 -> xyz=0 0 0.01365 rpy=2.1275 -1.5708 0
- joint camera_joint: origin xyz=0 0 0.049 rpy=0 0 0 -> xyz=0.011 0.044 0.013 rpy=0 0 0
- joint elbow_joint: axis 0 1 0 -> 0 0 1; limit lower=-1.5708 upper=1.5708 effort=5 velocity=3 -> lower=-3.075 upper=0.065 effort=5 velocity=3; origin xyz=0 0 0.1452 rpy=0 0.85 0 -> xyz=0.1452 -0.0001 0 rpy=3.1416 0 2.0591
- joint shoulder_joint: axis 0 1 0 -> 0 0 1; limit lower=-1.5708 upper=1.5708 effort=5 velocity=3 -> lower=-1.571 upper=0.05 effort=5 velocity=3; origin xyz=0 0 0.04137 rpy=0 0 0 -> xyz=0.04225 0 0 rpy=0 0 1.0414
- joint wrist_joint: axis 0 1 0 -> 0.074068 0 -0.99725; limit lower=-1.5708 upper=1.5708 effort=5 velocity=3 -> lower=-2.071 upper=1.0708 effort=5 velocity=3; origin xyz=0 0 0.1 rpy=0 0.25 0 -> xyz=0 -0.1 0 rpy=0 0.074136 2.2399

Commit message: Add calibrated Raspberry Pi control backend
Implement safe radians-to-PWM calibration and align simulation actions, configuration, documentation, and tests with the verified physical arm range.

Co-authored-by: Cursor <cursoragent@cursor.com>

File: models/butter_finger_simple.urdf (robot description, URDF)
Before this commit: robot butter_finger, 6 links, 5 joints
Joints:
- joint shoulder_joint: limit lower=-1.571 upper=0.05 effort=5 velocity=3 -> lower=-1.53 upper=0 effort=5 velocity=3
- joint wrist_joint: limit lower=-2.071 upper=1.0708 effort=5 velocity=3 -> lower=-2.9824 upper=0.1576 effort=5 velocity=3
